Commit message: Added zed model and ball detection

File: urdf/roverCool.urdf (robot description, URDF)
Before this commit: robot rover, 8 links, 7 joints
Links:
- added link zed_center; visual mesh filename=package://zed_wrapper/urdf/ZED.stl
- added link zed_depth_camera
- added link zed_left_camera; visual cylinder length=.031 radius=0.007
- added link zed_right_camera; visual cylinder length=.031 radius=0.007
Joints:
- added joint chasis_to_zed: type fixed, parent chasis, child zed_center, origin xyz=0.195  0 0
- added joint zed_depth_camera_joint: type fixed, parent zed_left_camera, child zed_depth_camera, origin xyz=0 0 0 rpy=-1.5707963267948966 0 -1.5707963267948966
- added joint zed_left_camera_joint: type fixed, parent zed_center, child zed_left_camera, origin xyz=0 0.06 0 rpy=0 0 0
- added joint zed_right_camera_joint: type fixed, parent zed_center, child zed_right_camera, origin xyz=0 -0.06 0 rpy=0 0 0
