Commit message: Added robotic arm model

File: urdf/completeRover.urdf (robot description, URDF)
Before this commit: robot rover, 14 links, 13 joints
Links:
- added link arm_base; visual mesh filename=package://model/meshes/arm1.STL scale=0.001 0.001 0.001
- added link elbow; visual mesh filename=package://model/meshes/arm2.STL scale=0.001 0.001 0.001
- added link forearm; visual mesh filename=package://model/meshes/arm3.STL scale=0.001 0.001 0.001
- added link rotation; visual mesh filename=package://model/meshes/rotate.STL scale=0.001 0.001 0.001
- added link wrist; visual mesh filename=package://model/meshes/UpDown.STL scale=0.001 0.001 0.001
Joints:
- added joint arm_to_wrist: type revolute, parent forearm, child wrist, origin xyz=0.285 0 0.1, axis 0 1 0, limit lower=-0.6 upper=0.6 effort=1000.0 velocity=.1
- added joint base: type revolute, parent chasis, child arm_base, origin xyz=0.20  0 0, axis 0 0 1, limit lower=-0.6 upper=0.6 effort=1000.0 velocity=.1
- added joint base_to_elbow: type revolute, parent arm_base, child elbow, origin xyz=0 0 0.115, axis 0 1 0, limit lower=-0.6 upper=0.6 effort=1000.0 velocity=.1
- added joint elbow_to_arm: type revolute, parent elbow, child forearm, origin xyz=0.32 0 0.11, axis 0 1 0, limit lower=-0.6 upper=0.6 effort=1000.0 velocity=.1
- added joint wrist_to_rotate: type revolute, parent wrist, child rotation, origin xyz=0 0 0.1, axis 0 1 0, limit lower=-0.6 upper=0.6 effort=1000.0 velocity=.1

Commit message: Added complet robotic arm

File: urdf/completeRover.urdf (robot description, URDF)
Before this commit: robot rover, 19 links, 18 joints
Links:
- added link finger; visual mesh filename=package://model/meshes/finger.STL scale=0.001 0.001 0.001
Joints:
- added joint rotate_to_finger: type prismatic, parent rotation, child finger, origin xyz=-0.06 0 0.095, axis 1 0 0, limit lower=0 upper=0.08 effort=1000.0 velocity=.1
- joint arm_to_wrist: limit lower=-0.6 upper=0.6 effort=1000.0 velocity=.1 -> lower=-3.1416 upper=3.1416 effort=1000.0 velocity=.1
- joint base_to_elbow: limit lower=-0.6 upper=0.6 effort=1000.0 velocity=.1 -> lower=-3.1416 upper=3.1416 effort=1000.0 velocity=.1
- joint elbow_to_arm: limit lower=-0.6 upper=0.6 effort=1000.0 velocity=.1 -> lower=-3.1416 upper=3.1416 effort=1000.0 velocity=.1
- joint wrist_to_rotate: axis 0 1 0 -> 0 0 1; limit lower=-0.6 upper=0.6 effort=1000.0 velocity=.1 -> lower=-3.1416 upper=3.1416 effort=1000.0 velocity=.1; origin xyz=0 0 0.1 -> xyz=0 0 0.055

File: urdf/robotArm.urdf (robot description, URDF)
Before this commit: robot rover, 6 links, 5 joints
Links:
- added link finger; visual mesh filename=package://model/meshes/finger.STL scale=0.001 0.001 0.001
Joints:
- added joint rotate_to_finger: type prismatic, parent rotation, child finger, origin xyz=-0.06 0 0.095, axis 1 0 0, limit lower=0 upper=0.08 effort=1000.0 velocity=.1
- joint arm_to_wrist: limit lower=-0.6 upper=0.6 effort=1000.0 velocity=.1 -> lower=-3.1416 upper=3.1416 effort=1000.0 velocity=.1
- joint base: limit lower=-0.6 upper=0.6 effort=1000.0 velocity=.1 -> lower=-3.1416 upper=3.1416 effort=1000.0 velocity=.1
- joint base_to_elbow: limit lower=-0.6 upper=0.6 effort=1000.0 velocity=.1 -> lower=-3.1416 upper=3.1416 effort=1000.0 velocity=.1
- joint elbow_to_arm: limit lower=-0.6 upper=0.6 effort=1000.0 velocity=.1 -> lower=-3.1416 upper=3.1416 effort=1000.0 velocity=.1
- joint wrist_to_rotate: axis 0 1 0 -> 0 0 1; limit lower=-0.6 upper=0.6 effort=1000.0 velocity=.1 -> lower=-3.1416 upper=3.1416 effort=1000.0 velocity=.1; origin xyz=0 0 0.1 -> xyz=0 0 0.055
